File: bsidesorl-v1/dc407-sao.kicad_pcb (KiCad board)
At the start: 2 copper layers, 39.5 x 23 mm, 7 parts

Commit message: added 561
Routing:
- net Net-(BT1-+): track 25.1 -> 25.6 mm
Changed lines of the file:
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@@
   (segment (start 147.523654 101.86) (end 148.703654 100.68) (width 0.2) (layer "B.Cu") (net 1))
   (segment (start 146.61 101.86) (end 147.523654 101.86) (width 0.2) (layer "B.Cu") (net 1))
-  (segment (start 152.58 97.89) (end 158.01 92.46) (width 0.2) (layer "B.Cu") (net 2))
-  (segment (start 148.04 97.89) (end 152.58 97.89) (width 0.2) (layer "B.Cu") (net 2))
+  (segment (start 148.04 97.89) (end 153.5 97.89) (width 0.2) (layer "B.Cu") (net 2))
+  (segment (start 153.5 97.89) (end 158.01 93.38) (width 0.2) (layer "B.Cu") (net 2))
+  (segment (start 139.2 93.48) (end 145.04 99.32) (width 0.2) (layer "B.Cu") (net 2))
+  (segment (start 158.01 93.38) (end 158.01 92.46) (width 0.2) (layer "B.Cu") (net 2))
+  (segment (start 139.2 92.46) (end 139.2 93.48) (width 0.2) (layer "B.Cu") (net 2))
   (segment (start 145.04 99.32) (end 146.61 99.32) (width 0.2) (layer "B.Cu") (net 2))
-  (segment (start 139.2 92.46) (end 139.2 93.48) (width 0.2) (layer "B.Cu") (net 2))
   (segment (start 146.61 99.32) (end 148.04 97.89) (width 0.2) (layer "B.Cu") (net 2))
-  (segment (start 139.2 93.48) (end 145.04 99.32) (width 0.2) (layer "B.Cu") (net 2))
 )
