File: bsidesorl-v1/iwc-iron-sao.kicad_pcb (KiCad board)
At the start: 2 copper layers, 29.6 x 32 mm, 4 parts

Commit message: added 561
Parts:
- moved G*** 2.67 mm to (152.6, 108.1)
Other:
- board size 29.6 x 32 mm -> 37.9 x 41 mm
